File: PCB/Power.kicad_sch (KiCad schematic)
At the start: 70 parts

Commit message: Sch in progress, eMMC added
Parts:
- removed C?: 0.1u, Capacitors:CAP_0402, symbol Tittar_kl:C
- removed L? (x5): 1uH, Inductors:IND_SRN2512, symbol Tittar_kl:L
- removed R?: 1k, Resistors:RES_0402_sm, symbol Tittar_kl:R
- removed SW?: BUTTON, symbol Switches:BUTTON
- added C? (x2): 1u, Capacitors:CAP_0603, symbol Tittar_kl:C
- added C? (x2): 10u, Capacitors:CAP_0603, symbol Tittar_kl:C
- added C? (x2): 100uF, Capacitors:CAP_1206, symbol Tittar_kl:C
- added D?: PMEG2020, Diodes:SOD323, symbol Tittar_kl:D_Shottky
- added DA?: LPW5210, SOT:SOT23-5, symbol Power_kl:LPW5210
- added DA?: MT3608, SOT:SOT23-6, symbol Power_kl:MT3608
- added L?: 2.2uH, Inductors:IND_SRN2512, symbol Tittar_kl:L
- added L? (x5): 1uH, Inductors:IND_SRN2512, symbol Tittar_kl:L
- added R? (x2): 0R, Resistors:RES_0402_sm, symbol Tittar_kl:R
- added R? (x2): 10k, Resistors:RES_0402_sm, symbol Tittar_kl:R
- added R?: 130k, Resistors:RES_0402_sm, symbol Tittar_kl:R
- added R?: 1M, Resistors:RES_0402_sm, symbol Tittar_kl:R
- C? (x14): footprint Capacitors:CAP_0402 -> Capacitors:CAP_0603; Voltage (none) -> 10V
- C? (x27): Voltage (none) -> 10V
- L?: PN SRN2512-1R0M -> SRP2512-1R0M; Price 9 -> 14; URL https://www.terraelectronica.ru/product/1638188 -> https://www.terraelectronica.ru/product/1638486
- R?: footprint Resistors:RES_0805 -> Resistors:RES_0603
Connections:
- net GND: now also C?.2, C?.2, C?.2, C?.2, C?.2, C?.2, DA?.2 (GND), DA?.2 (GND), R?.1, R?.1; no longer DA?.12 (GND), DA?.25 (GND), DA?.45 (GND), DA?.59 (GND), DA?.69 (GND)
- net IPS: no longer C?.1, C?.1, C?.1, C?.1, C?.1, C?.1, C?.1, DA?.11 (VIN6), DA?.19 (VIN1), DA?.32 (ALDOIN), DA?.38 (VIN3), DA?.39 (VIN2), DA?.40 (VIN2), DA?.55 (IPSOUT), DA?.56 (IPSOUT), DA?.66 (VIN_CHG), Q?.1 (S), Q?.2 (S), Q?.3 (S)
- net VBAT: no longer C?.1, C?.1, DA?.64 (BATSENSE), R?.1
- net LDSNS: now reaches C?.1, C?.1, C?.2, DA?.63 (LOADSENSE), Q?.5 (D), Q?.6 (D), Q?.7 (D), Q?.8 (D), R?.2
- net LDSNS: now also L?.2
- net at DA?.65 (LX_CHG): now also L?.1
- net LX6: now reaches DA?.10 (LX6)
- net LX6: now also L?.1
- net LX3: now reaches DA?.36 (LX3), DA?.37 (LX3)
- net LX3: now also L?.1
- net LX1: now reaches DA?.21 (LX1)
- net LX1: now also L?.1
- net LX2: now reaches DA?.43 (LX2), DA?.44 (LX2)
- net LX2: now also L?.1
- net AP_RESET: now reaches DA?.46 (PWROK)
- net AP_NMI: now reaches DA?.61 (IRQ)
- net AP_NMI: now also R?.1
- net LX5: now reaches DA?.7 (LX5), L?.1
- net DDR1v2 renamed +VCC_DRAM
- net DLDO1 renamed +VCC3V3VID
- net ELDO1 renamed +VDD1V8
- net PMU-SCK renamed PMU.SCK
- net PMU-SDA renamed PMU.SDA
- net PWRON renamed BTN_PWRON
- net USB0-DM renamed USB0.DM
- net USB0-DP renamed USB0.DP
- net VCC-IO renamed +VCCIO3V3
- net +VCCIO3V3: now also L?.2, R?.2
- net VCC-PL renamed +VCCPL1V8
- net VCC-PLL renamed +AVCCPLL
- net VCC-RTC renamed +VCCRTC
- net +VCCRTC: now also R?.2
- net VCC1v2-HSIC renamed +VCC1V2HSIC
- net VDD-CPUS renamed +VDDCPUS1V1
- net VDD-CPUX renamed +VDDCPUX
- net +VDDCPUX: now also L?.2, L?.2
- net VDD-SYS renamed +VDDSYS1V1
- net +VDDSYS1V1: now also L?.2
- new net: DA?.3 (RSET), R?.2
- new net: DA?.3 (FB), R?.1, R?.2
- new net +5V: C?.1, C?.1, D?.C, DA?.4 (EN), DA?.5 (VIN), R?.1, R?.2
- new net +IPS: C?.1, C?.1, C?.1, C?.1, C?.1, C?.1, C?.1, C?.1, C?.1, C?.1, DA?.11 (VIN6), DA?.19 (VIN1), DA?.32 (ALDOIN), DA?.38 (VIN3), DA?.39 (VIN2), DA?.40 (VIN2), DA?.5 (IN), DA?.55 (IPSOUT), DA?.56 (IPSOUT), DA?.66 (VIN_CHG), L?.2, Q?.1 (S), Q?.2 (S), Q?.3 (S)
- new net +USBVOUT: C?.1, DA?.1 (VOUT), R?.2
- new net +VBAT: C?.1, C?.1, DA?.64 (BATSENSE), R?.1
- new net 5VEN: DA?.4 (EN), R?.1
- new net LX5V: D?.A, DA?.1 (LX), L?.1
Other:
- note added: "Mount if 5V control is not required"
- note added: "Mount if protection is not required"
- moved on the sheet: C?, DA?A, DA?B, DA?C, DA?D, DA?E, DA?F, DA?G, DA?H, DA?I, DA?J, DA?K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

Commit message: + LCD
Parts:
- gave numbers to parts that had none: 1
Connections:
- net USB_VBUS is gone; now on net +USBVIN: C?.1, C?.1, DA1.54 (VBUS), DA1.57 (ACIN), DA1.58 (ACIN)
Changed lines of the file:
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@@
     (stroke (width 0) (type solid) (color 0 0 0 0))
   )
+  (wire (pts (xy 33.02 213.36) (xy 48.26 213.36))
+    (stroke (width 0) (type default) (color 0 0 0 0))
+  )
   (wire (pts (xy 57.15 175.26) (xy 68.58 175.26))
     (stroke (width 0) (type default) (color 0 0 0 0))
@@
     (effects (font (size 1.27 1.27)) (justify left bottom))
   )
+  (label "+IPS" (at 48.26 213.36 180)
+    (effects (font (size 1.27 1.27)) (justify right bottom))
+  )
   (label "+VDD1V8" (at 48.26 242.57 180)
     (effects (font (size 1.27 1.27)) (justify right bottom))
@@
     (effects (font (size 1.27 1.27)) (justify left bottom))
   )
+  (label "+USBVIN" (at 82.55 30.48 0)
+    (effects (font (size 1.27 1.27)) (justify left bottom))
+  )
   (label "+VDDSYS1V1" (at 48.26 219.71 180)
     (effects (font (size 1.27 1.27)) (justify right bottom))
@@
     (effects (font (size 1.27 1.27)) (justify left bottom))
   )
-  (label "USB_VBUS" (at 82.55 30.48 0)
-    (effects (font (size 1.27 1.27)) (justify left bottom))
-  )
   (label "VINT" (at 119.38 170.18 180)
     (effects (font (size 1.27 1.27)) (justify right bottom))
@@
     (effects (font (size 1.27 1.27)) (justify right))
   )
+  (hierarchical_label "+IPS" (shape output) (at 33.02 213.36 180)
+    (effects (font (size 1.27 1.27)) (justify right))
+  )
   (hierarchical_label "AP_RESET" (shape output) (at 128.27 157.48 0)
     (effects (font (size 1.27 1.27)) (justify left))
@@
   (symbol (lib_id "Power_kl:AXP803") (at 71.12 88.9 0) (mirror y) (unit 12)
     (in_bom yes) (on_board yes)
-    (property "Reference" "DA?" (id 0) (at 67.31 80.01 0)
+    (property "Reference" "DA1" (id 0) (at 67.31 80.01 0)
       (effects (font (size 1.27 1.27)) (justify left))
     )
@@
   (symbol (lib_name "AXP803_3") (lib_id "Power_kl:AXP803") (at 252.73 99.06 0) (unit 3)
     (in_bom yes) (on_board yes)
-    (property "Reference" "DA?" (id 0) (at 247.65 91.44 0))
+    (property "Reference" "DA1" (id 0) (at 247.65 91.44 0))
     (property "Value" "AXP803" (id 1) (at 256.54 91.44 0))
     (property "Footprint" "QFN_DFN:QFN-68_EP_8x8_Pitch0.4mm" (id 2) (at 252.73 92.71 0)
@@
   (symbol (lib_id "Power_kl:AXP803") (at 251.46 34.29 0) (unit 1)
     (in_bom yes) (on_board yes)
-    (property "Reference" "DA?" (id 0) (at 246.38 26.67 0))
+    (property "Reference" "DA1" (id 0) (at 246.38 26.67 0))
     (property "Value" "AXP803" (id 1) (at 256.54 26.67 0))
     (property "Footprint" "QFN_DFN:QFN-68_EP_8x8_Pitch0.4mm" (id 2) (at 251.46 27.94 0)
@@
   (symbol (lib_name "AXP803_4") (lib_id "Power_kl:AXP803") (at 266.7 265.43 0) (unit 14)
     (in_bom yes) (on_board yes)
-    (property "Reference" "DA?" (id 0) (at 270.51 254 0))
+    (property "Reference" "DA1" (id 0) (at 270.51 254 0))
     (property "Value" "AXP803" (id 1) (at 270.51 256.54 0))
     (property "Footprint" "QFN_DFN:QFN-68_EP_8x8_Pitch0.4mm" (id 2) (at 266.7 259.08 0)
@@
   (symbol (lib_id "Power_kl:AXP803") (at 168.91 71.12 0) (unit 8)
     (in_bom yes) (on_board yes)
-    (property "Reference" "DA?" (id 0) (at 172.72 59.69 0))
+    (property "Reference" "DA1" (id 0) (at 172.72 59.69 0))
     (property "Value" "AXP803" (id 1) (at 172.72 62.23 0))
     (property "Footprint" "QFN_DFN:QFN-68_EP_8x8_Pitch0.4mm" (id 2) (at 168.91 64.77 0)
@@
   (symbol (lib_name "AXP803_2") (lib_id "Power_kl:AXP803") (at 250.19 129.54 0) (unit 4)
     (in_bom yes) (on_board yes)
-    (property "Reference" "DA?" (id 0) (at 246.38 121.92 0))
+    (property "Reference" "DA1" (id 0) (at 246.38 121.92 0))
     (property "Value" "AXP803" (id 1) (at 256.54 121.92 0))
     (property "Footprint" "QFN_DFN:QFN-68_EP_8x8_Pitch0.4mm" (id 2) (at 250.19 123.19 0)
@@
   (symbol (lib_name "AXP803_13") (lib_id "Power_kl:AXP803") (at 252.73 67.31 0) (unit 2)
     (in_bom yes) (on_board yes)
-    (property "Reference" "DA?" (id 0) (at 246.38 58.42 0))
+    (property "Reference" "DA1" (id 0) (at 246.38 58.42 0))
     (property "Value" "AXP803" (id 1) (at 256.54 58.42 0))
     (property "Footprint" "QFN_DFN:QFN-68_EP_8x8_Pitch0.4mm" (id 2) (at 252.73 60.96 0)
@@
   (symbol (lib_name "AXP803_5") (lib_id "Power_kl:AXP803") (at 251.46 189.23 0) (unit 6)
     (in_bom yes) (on_board yes)
-    (property "Reference" "DA?" (id 0) (at 255.27 177.8 0))
+    (property "Reference" "DA1" (id 0) (at 255.27 177.8 0))
     (property "Value" "AXP803" (id 1) (at 255.27 180.34 0))
     (property "Footprint" "QFN_DFN:QFN-68_EP_8x8_Pitch0.4mm" (id 2) (at 251.46 182.88 0)
@@
   (symbol (lib_id "Power_kl:AXP803") (at 170.18 110.49 0) (unit 10)
     (in_bom yes) (on_board yes)
-    (property "Reference" "DA?" (id 0) (at 173.99 97.79 0))
+    (property "Reference" "DA1" (id 0) (at 173.99 97.79 0))
     (property "Value" "AXP803" (id 1) (at 173.99 100.33 0))
     (property "Footprint" "QFN_DFN:QFN-68_EP_8x8_Pitch0.4mm" (id 2) (at 170.18 104.14 0)
@@
   (symbol (lib_id "Power_kl:AXP803") (at 87.63 158.75 0) (unit 13)
     (in_bom yes) (on_board yes)
-    (property "Reference" "DA?" (id 0) (at 88.9 147.32 0))
+    (property "Reference" "DA1" (id 0) (at 88.9 147.32 0))
     (property "Value" "AXP803" (id 1) (at 88.9 149.86 0))
     (property "Footprint" "QFN_DFN:QFN-68_EP_8x8_Pitch0.4mm" (id 2) (at 87.63 152.4 0)
@@
   (symbol (lib_id "Power_kl:AXP803") (at 167.64 151.13 0) (unit 9)
     (in_bom yes) (on_board yes)
-    (property "Reference" "DA?" (id 0) (at 172.72 139.7 0))
+    (property "Reference" "DA1" (id 0) (at 172.72 139.7 0))
     (property "Value" "AXP803" (id 1) (at 172.72 142.24 0))
     (property "Footprint" "QFN_DFN:QFN-68_EP_8x8_Pitch0.4mm" (id 2) (at 167.64 144.78 0)
@@
   (symbol (lib_id "Power_kl:AXP803") (at 168.91 35.56 0) (unit 7)
     (in_bom yes) (on_board yes)
-    (property "Reference" "DA?" (id 0) (at 172.72 22.86 0))
+    (property "Reference" "DA1" (id 0) (at 172.72 22.86 0))
     (property "Value" "AXP803" (id 1) (at 172.72 25.4 0))
     (property "Footprint" "QFN_DFN:QFN-68_EP_8x8_Pitch0.4mm" (id 2) (at 168.91 29.21 0)
@@
   (symbol (lib_id "Power_kl:AXP803") (at 120.65 35.56 0) (unit 11)
     (in_bom yes) (on_board yes)
-    (property "Reference" "DA?" (id 0) (at 113.03 26.67 0)
+    (property "Reference" "DA1" (id 0) (at 113.03 26.67 0)
       (effects (font (size 1.27 1.27)) (justify left))
     )
@@
   (symbol (lib_name "AXP803_1") (lib_id "Power_kl:AXP803") (at 251.46 153.67 0) (unit 5)
     (in_bom yes) (on_board yes)
-    (property "Reference" "DA?" (id 0) (at 246.38 144.78 0))
+    (property "Reference" "DA1" (id 0) (at 246.38 144.78 0))
     (property "Value" "AXP803" (id 1) (at 256.54 144.78 0))
     (property "Footprint" "QFN_DFN:QFN-68_EP_8x8_Pitch0.4mm" (id 2) (at 251.46 147.32 0)
