File: PCB/CPU.kicad_sch (KiCad schematic)
At the start: 0 parts

Commit message: Sch in progress, eMMC added
Parts:
- added C? (x8): 1u, Capacitors:CAP_0402, symbol Tittar_kl:C
- added C? (x21): 0u1, Capacitors:CAP_0402, symbol Tittar_kl:C
- added C? (x2): 2u2, Capacitors:CAP_0402, symbol Tittar_kl:C
- added C? (x5): 4u7, Capacitors:CAP_0402, symbol Tittar_kl:C
- added C? (x7): 10u, Capacitors:CAP_0603, symbol Tittar_kl:C
- added C? (x2): 18pF, Capacitors:CAP_0402, symbol Tittar_kl:C
- added C? (x2): 6.8pF, Capacitors:CAP_0402, symbol Tittar_kl:C
- added C?: 10nF, Capacitors:CAP_0402, symbol Tittar_kl:C
- added C?: 1nF, Capacitors:CAP_0402, symbol Tittar_kl:C
- added DD1: A64, BGA:BGA-529_23x23_15.0x15.0mm, symbol Allwinner:A64
- added F?: Fuse0R, PCB:FuseShorted, symbol Tittar_kl:Fuse0R
- added R?: 33R, Resistors:RES_0402_sm, symbol Tittar_kl:R
- added R?: 56k, Resistors:RES_0402_sm, symbol Tittar_kl:R
- added R? (x2): 1k, Resistors:RES_0402_sm, symbol Tittar_kl:R
- added R?: 200k, Resistors:RES_0402_sm, symbol Tittar_kl:R
- added R?: 10M, Resistors:RES_0402_sm, symbol Tittar_kl:R
- added R?: 20k, Resistors:RES_0402_sm, symbol Tittar_kl:R
- added R? (x2): 100k, Resistors:RES_0402_sm, symbol Tittar_kl:R
- added SW? (x3): IT1198, BtnsSwitches:BTN_IT1198, symbol BtnsSwitches:BUTTON
- added SW?: BUTTON, BtnsSwitches:BTN_4x4_SMD, symbol BtnsSwitches:BUTTON
- added TP?: TESTPOINT, PCB:TESTPOINT_1MM, symbol pcb_details:TESTPOINT
- added XTAL?: 24MHz, Quartz:03225C4, symbol Tittar_kl:CRYSTAL_H
- added XTAL?: 32768, Quartz:03215C2, symbol Tittar_kl:CRYSTAL
Connections:
- net GND: now also C?.1, C?.1, C?.1, C?.1, C?.1, C?.2, C?.2, C?.2, C?.2, C?.2, C?.2, C?.2, C?.2, C?.2, C?.2, C?.2, C?.2, C?.2, C?.2, C?.2, C?.2, C?.2, C?.2, C?.2, C?.2, C?.2, C?.2, C?.2, C?.2, C?.2, C?.2, C?.2, C?.2, C?.2, C?.2, C?.2, C?.2, C?.2, C?.2, C?.2, C?.2, C?.2, DD1.A1 (GND), DD1.A23 (GND), DD1.AC23 (GND), DD1.C3 (GND), DD1.C7 (GND), DD1.D7 (GND), DD1.G11 (GND), DD1.G6 (GND), DD1.H13 (GND), DD1.H4 (GND), DD1.J10 (GND), DD1.J11 (GND), DD1.J14 (GND), DD1.J15 (GND), DD1.J9 (GND), DD1.K10 (GND), DD1.K11 (GND), DD1.K12 (GND), DD1.K13 (GND), DD1.K8 (GND), DD1.K9 (GND), DD1.L10 (GND), DD1.L11 (GND), DD1.L12 (GND), DD1.L15 (GND), DD1.L4 (GND), DD1.L5 (GND), DD1.L9 (GND), DD1.M10 (GND), DD1.M11 (GND), DD1.M12 (GND), DD1.M15 (GND), DD1.M3 (GND), DD1.M8 (GND), DD1.M9 (GND), DD1.N10 (GND), DD1.N11 (GND), DD1.N12 (GND), DD1.N13 (GND), DD1.N15 (GND), DD1.N4 (GND), DD1.N9 (GND), DD1.P10 (GND), DD1.P11 (GND), DD1.P12 (GND), DD1.P13 (GND), DD1.P7 (GND), DD1.P8 (GND), DD1.P9 (GND), DD1.R10 (GND), DD1.R11 (GND), DD1.R12 (GND), DD1.R15 (GND), DD1.R5 (GND), DD1.R6 (GND), DD1.R7 (GND), DD1.R8 (GND), DD1.R9 (GND), DD1.T10 (GND), DD1.T11 (GND), DD1.T12 (GND), DD1.T13 (GND), DD1.T8 (GND), DD1.T9 (GND), DD1.U11 (GND), DD1.U12 (GND), DD1.U2 (GND), DD1.U5 (GND), DD1.U7 (GND), DD1.U8 (GND), DD1.U9 (GND), DD1.V14 (GND), DD1.V8 (GND), F?.2, R?.1, SW?.2, SW?.2, SW?.2, SW?.2, XTAL?.H
- new net: DD1.B18 (X32KFOUT), R?.2
- new net: R?.1, SW?.1 (x4)
- new net: C?.1, DD1.P16 (VDDBP-EFUSE)
- new net: C?.1, DD1.G16 (RTC-VIO)
- new net: C?.1, DD1.E10 (CPN)
- new net: C?.2, DD1.E11 (CPP)
- new net +AVCCPLL: C?.1, C?.1, C?.2, DD1.G14 (AVCC), DD1.N16 (VCC-PLL), R?.2
- new net +VCC1V2HSIC: C?.2, DD1.K16 (HSIC-VCC)
- new net +VCC3V3VID: C?.1, C?.1, DD1.M16 (HVCC), DD1.N19 (VCC-DSI)
- new net +VCCIO3V3: C?.1, C?.1, C?.1, C?.1, C?.2, DD1.L16 (VCC-USB), DD1.N18 (VCC-EFUSE), DD1.T14 (VCC-IO), DD1.U15 (VCC-IO)
- new net +VCCPL1V8: C?.1, DD1.J16 (VCC-PL)
- new net +VCCRTC: C?.1, C?.1, DD1.H16 (VCC-RTC)
- new net +VDD1V8: C?.1, C?.2, DD1.E13 (CPVDD)
- new net +VDDCPUS1V1: C?.1, C?.1, DD1.H15 (VDD-CPUS)
- new net +VDDCPUX: C?.1, C?.1, C?.1, C?.1, C?.1, C?.1, C?.1, C?.1, C?.1, DD1.AA1 (VDD-CPUX), DD1.AA3 (VDD-CPUX), DD1.AB2 (VDD-CPUX), DD1.AC1 (VDD-CPUX), DD1.AC2 (VDD-CPUX), DD1.U6 (VDD-CPUX), DD1.V2 (VDD-CPUX), DD1.V3 (VDD-CPUX), DD1.V4 (VDD-CPUX), DD1.V5 (VDD-CPUX), DD1.V6 (VDD-CPUX), DD1.W1 (VDD-CPUX), DD1.W3 (VDD-CPUX), DD1.W4 (VDD-CPUX), DD1.W5 (VDD-CPUX), DD1.Y2 (VDD-CPUX), DD1.Y3 (VDD-CPUX), DD1.Y4 (VDD-CPUX)
- new net +VDDSYS1V1: C?.1, C?.1, C?.1, C?.1, C?.1, DD1.J12 (VDD-SYS), DD1.J13 (VDD-SYS), DD1.K14 (VDD-SYS), DD1.L13 (VDD-SYS), DD1.L14 (VDD-SYS), DD1.M13 (VDD-SYS), DD1.M14 (VDD-SYS), DD1.N14 (VDD-SYS), DD1.P14 (VDD-SYS), DD1.R13 (VDD-SYS), DD1.R14 (VDD-SYS), DD1.T15 (VDD-SYS)
- new net 5VEN: DD1.D22 (PL12), R?.2
- new net AGND: C?.1, C?.1, C?.1, C?.2, C?.2, C?.2, DD1.A11 (AGND), F?.1, R?.1
- new net AP_CK32KO: R?.1
- new net AP_NMI: C?.1, DD1.G18 (NMI)
- new net AP_RESET: C?.1, DD1.E17 (RESET), R?.2
- new net AP_WAKE_BT: DD1.B20 (PL6/S-JTAG-DO)
- new net BTN_PWRON: C?.1, R?.2
- new net BT_REG_ON: DD1.A20 (PL4/S-JTAG-MS)
- new net BT_WAKE_AP: DD1.D19 (PL5/S-JTAG-CK)
- new net CPVEE: C?.1, C?.1, DD1.F12 (CPVEE), DD1.G13 (VEE)
- new net KEYADC: C?.1, DD1.A16 (KEYADC), R?.1, R?.2, R?.2
- new net LCD_PWM: DD1.D21 (PL10/S-PWM)
- new net PMU.SCK: DD1.D17 (PL0/S-RSB-SCK/S-TWI-SCK)
- new net PMU.SDA: DD1.C17 (PL1/S-RSB-SDA/S-TWI-SDA)
- new net UBOOT: DD1.F17 (FEL), TP?.1
- new net USB0.DM: DD1.B22 (USB0-DM)
- new net USB0.DP: DD1.A22 (USB0-DP)
- new net USB1.DM: DD1.C22 (USB1-DM)
- new net USB1.DP: DD1.B23 (USB1-DP)
- new net VDDFB-CPUX: DD1.T6 (VDDFB-CPUX)
- new net VRA1: C?.2, DD1.B12 (VRA1)
- new net VRA2: C?.1, DD1.B11 (VRA2), R?.2
- new net VRP: C?.1, C?.2, DD1.C11 (VRP)
- new net WL_REG_ON: DD1.A19 (PL2/S-UART-TX)
- new net WL_WAKE_AP: DD1.E19 (PL3/S-UART-RX)
- new net X24MI: C?.1, DD1.K22 (X24MI), XTAL?.1
- new net X24MO: C?.1, DD1.K23 (X24MO), XTAL?.2
- new net X32KI: C?.2, DD1.C18 (X32KIN), R?.1, XTAL?.1
- new net X32KO: C?.2, DD1.B19 (X32KOUT), R?.2, XTAL?.2
- no-connect marks 0 -> 52
Other:
- note added: "AUDIO"
- note added: "HDMI + MIPI"
- note added: "PwrOn"
- note added: "RESET"
- note added: "Volume Up/Down"

Commit message: + LCD
Parts:
- removed C? (x2): 0u1, Capacitors:CAP_0402, symbol Tittar_kl:C
- removed unit 4 of DD1
- added C?: 4u7, Capacitors:CAP_0402, symbol Tittar_kl:C
- added unit 9 of DD1
- added DD? (x6): A64, BGA:BGA-529_23x23_15.0x15.0mm, symbol Allwinner:A64
Connections:
- net +VCCIO3V3: now also C?.1, DD1.U18 (VCC-PE)
- net GND: now also C?.2
- net LCD_PWM: no longer names the net of DD1.D21 (PL10/S-PWM)
- no-connect marks 52 -> 68
Other:
- note added: "POWER"
- note added: "SYS & WL/BT"
- moved on the sheet: C?, DD1B, DD1L, R?, SW?, TP?

Commit message: Before eMMC removing
Parts:
- removed DD? (x5): A64, BGA:BGA-529_23x23_15.0x15.0mm, symbol Allwinner:A64
- added unit 13 of DD1
- added unit 14 of DD1
- added XL?: CONN_3, Connectors:PLS-3, symbol Connectors_kl:CONN_3
- gave numbers to parts that had none: 1
Connections:
- net +VCCIO3V3: now also DD1.T14 (VCC-IO), DD1.U15 (VCC-IO); no longer DD1.T14 (VCC-IO), DD1.U15 (VCC-IO)
- net +VCCPL1V8: now also DD1.J16 (VCC-PL); no longer DD1.J16 (VCC-PL)
- net +VDDCPUS1V1: now also DD1.H15 (VDD-CPUS); no longer DD1.H15 (VDD-CPUS)
- net +VDDCPUX: now also DD1.AA1 (VDD-CPUX), DD1.AA3 (VDD-CPUX), DD1.AB2 (VDD-CPUX), DD1.AC1 (VDD-CPUX), DD1.AC2 (VDD-CPUX), DD1.U6 (VDD-CPUX), DD1.V2 (VDD-CPUX), DD1.V3 (VDD-CPUX), DD1.V4 (VDD-CPUX), DD1.V5 (VDD-CPUX), DD1.V6 (VDD-CPUX), DD1.W1 (VDD-CPUX), DD1.W3 (VDD-CPUX), DD1.W4 (VDD-CPUX), DD1.W5 (VDD-CPUX), DD1.Y2 (VDD-CPUX), DD1.Y3 (VDD-CPUX), DD1.Y4 (VDD-CPUX); no longer DD1.AA1 (VDD-CPUX), DD1.AA3 (VDD-CPUX), DD1.AB2 (VDD-CPUX), DD1.AC1 (VDD-CPUX), DD1.AC2 (VDD-CPUX), DD1.U6 (VDD-CPUX), DD1.V2 (VDD-CPUX), DD1.V3 (VDD-CPUX), DD1.V4 (VDD-CPUX), DD1.V5 (VDD-CPUX), DD1.V6 (VDD-CPUX), DD1.W1 (VDD-CPUX), DD1.W3 (VDD-CPUX), DD1.W4 (VDD-CPUX), DD1.W5 (VDD-CPUX), DD1.Y2 (VDD-CPUX), DD1.Y3 (VDD-CPUX), DD1.Y4 (VDD-CPUX)
- net +VDDSYS1V1: now also DD1.J12 (VDD-SYS), DD1.J13 (VDD-SYS), DD1.K14 (VDD-SYS), DD1.L13 (VDD-SYS), DD1.L14 (VDD-SYS), DD1.M13 (VDD-SYS), DD1.M14 (VDD-SYS), DD1.N14 (VDD-SYS), DD1.P14 (VDD-SYS), DD1.R13 (VDD-SYS), DD1.R14 (VDD-SYS), DD1.T15 (VDD-SYS); no longer DD1.J12 (VDD-SYS), DD1.J13 (VDD-SYS), DD1.K14 (VDD-SYS), DD1.L13 (VDD-SYS), DD1.L14 (VDD-SYS), DD1.M13 (VDD-SYS), DD1.M14 (VDD-SYS), DD1.N14 (VDD-SYS), DD1.P14 (VDD-SYS), DD1.R13 (VDD-SYS), DD1.R14 (VDD-SYS), DD1.T15 (VDD-SYS)
- net 5VEN: now also DD1.D22 (PL12); no longer DD1.D22 (PL12)
- net AP_WAKE_BT: now also DD1.B20 (PL6/S-JTAG-DO); no longer DD1.B20 (PL6/S-JTAG-DO)
- net BT_REG_ON: now also DD1.A20 (PL4/S-JTAG-MS); no longer DD1.A20 (PL4/S-JTAG-MS)
- net BT_WAKE_AP: now also DD1.D19 (PL5/S-JTAG-CK); no longer DD1.D19 (PL5/S-JTAG-CK)
- net GND: now also DD1.A1 (GND), DD1.A23 (GND), DD1.AC23 (GND), DD1.C3 (GND), DD1.C7 (GND), DD1.D7 (GND), DD1.G11 (GND), DD1.G6 (GND), DD1.H13 (GND), DD1.H4 (GND), DD1.J10 (GND), DD1.J11 (GND), DD1.J14 (GND), DD1.J15 (GND), DD1.J9 (GND), DD1.K10 (GND), DD1.K11 (GND), DD1.K12 (GND), DD1.K13 (GND), DD1.K8 (GND), DD1.K9 (GND), DD1.L10 (GND), DD1.L11 (GND), DD1.L12 (GND), DD1.L15 (GND), DD1.L4 (GND), DD1.L5 (GND), DD1.L9 (GND), DD1.M10 (GND), DD1.M11 (GND), DD1.M12 (GND), DD1.M15 (GND), DD1.M3 (GND), DD1.M8 (GND), DD1.M9 (GND), DD1.N10 (GND), DD1.N11 (GND), DD1.N12 (GND), DD1.N13 (GND), DD1.N15 (GND), DD1.N4 (GND), DD1.N9 (GND), DD1.P10 (GND), DD1.P11 (GND), DD1.P12 (GND), DD1.P13 (GND), DD1.P7 (GND), DD1.P8 (GND), DD1.P9 (GND), DD1.R10 (GND), DD1.R11 (GND), DD1.R12 (GND), DD1.R15 (GND), DD1.R5 (GND), DD1.R6 (GND), DD1.R7 (GND), DD1.R8 (GND), DD1.R9 (GND), DD1.T10 (GND), DD1.T11 (GND), DD1.T12 (GND), DD1.T13 (GND), DD1.T8 (GND), DD1.T9 (GND), DD1.U11 (GND), DD1.U12 (GND), DD1.U2 (GND), DD1.U5 (GND), DD1.U7 (GND), DD1.U8 (GND), DD1.U9 (GND), DD1.V14 (GND), DD1.V8 (GND), XL?.1 (P1); no longer DD1.A1 (GND), DD1.A23 (GND), DD1.AC23 (GND), DD1.C3 (GND), DD1.C7 (GND), DD1.D7 (GND), DD1.G11 (GND), DD1.G6 (GND), DD1.H13 (GND), DD1.H4 (GND), DD1.J10 (GND), DD1.J11 (GND), DD1.J14 (GND), DD1.J15 (GND), DD1.J9 (GND), DD1.K10 (GND), DD1.K11 (GND), DD1.K12 (GND), DD1.K13 (GND), DD1.K8 (GND), DD1.K9 (GND), DD1.L10 (GND), DD1.L11 (GND), DD1.L12 (GND), DD1.L15 (GND), DD1.L4 (GND), DD1.L5 (GND), DD1.L9 (GND), DD1.M10 (GND), DD1.M11 (GND), DD1.M12 (GND), DD1.M15 (GND), DD1.M3 (GND), DD1.M8 (GND), DD1.M9 (GND), DD1.N10 (GND), DD1.N11 (GND), DD1.N12 (GND), DD1.N13 (GND), DD1.N15 (GND), DD1.N4 (GND), DD1.N9 (GND), DD1.P10 (GND), DD1.P11 (GND), DD1.P12 (GND), DD1.P13 (GND), DD1.P7 (GND), DD1.P8 (GND), DD1.P9 (GND), DD1.R10 (GND), DD1.R11 (GND), DD1.R12 (GND), DD1.R15 (GND), DD1.R5 (GND), DD1.R6 (GND), DD1.R7 (GND), DD1.R8 (GND), DD1.R9 (GND), DD1.T10 (GND), DD1.T11 (GND), DD1.T12 (GND), DD1.T13 (GND), DD1.T8 (GND), DD1.T9 (GND), DD1.U11 (GND), DD1.U12 (GND), DD1.U2 (GND), DD1.U5 (GND), DD1.U7 (GND), DD1.U8 (GND), DD1.U9 (GND), DD1.V14 (GND), DD1.V8 (GND)
- net PMU.SCK: now also DD1.D17 (PL0/S-RSB-SCK/S-TWI-SCK); no longer DD1.D17 (PL0/S-RSB-SCK/S-TWI-SCK)
- net PMU.SDA: now also DD1.C17 (PL1/S-RSB-SDA/S-TWI-SDA); no longer DD1.C17 (PL1/S-RSB-SDA/S-TWI-SDA)
- net VDDFB-CPUX: now also DD1.T6 (VDDFB-CPUX); no longer DD1.T6 (VDDFB-CPUX)
- net WL_REG_ON: now also DD1.A19 (PL2/S-UART-TX); no longer DD1.A19 (PL2/S-UART-TX)
- net WL_WAKE_AP: now also DD1.E19 (PL3/S-UART-RX); no longer DD1.E19 (PL3/S-UART-RX)
- net TX0: now reaches DD1.V10 (PB8/UART0-TX)
- net TX0: now also XL?.2 (PM)
- net RX0: now reaches DD1.Y7 (PB9/UART0-RX)
- net RX0: now also XL?.3
- no-connect marks 68 -> 75
Other:
- note added: "DBG UART"
- moved on the sheet: C?, DD1F, DD1I, R?, TP?, XTAL?
