File: PCB/LCD.kicad_sch (KiCad schematic)
At the start: 0 parts

Commit message: + LCD
Parts:
- added C?: 10u, Capacitors:CAP_0603, symbol Tittar_kl:C
- added C? (x3): 0u1, Capacitors:CAP_0402, symbol Tittar_kl:C
- added C?: 4u7, Capacitors:CAP_0805, symbol Tittar_kl:C
- added D?: PMEG4005, Diodes:SOD323, symbol Tittar_kl:D_Shottky
- added DA?: PT4110, SOT:SOT89-5, symbol Power_kl:PT4110
- added DD1: A64, BGA:BGA-529_23x23_15.0x15.0mm, symbol Allwinner:A64
- added L?: 10uH, Inductors:IND_1210_LQH32C, symbol Tittar_kl:L
- added L?: BLM15AG102SN1, Inductors:IND_0402, symbol Tittar_kl:L
- added R?: 20R, Resistors:RES_0603, symbol Tittar_kl:R
- added R?: 100k, Resistors:RES_0603, symbol Tittar_kl:R
- added TP? (x6): TESTPOINT, PCB:TESTPOINT_1MM, symbol pcb_details:TESTPOINT
- added XL?: CONN_40, Connectors:FFC_0d5x40_flip, symbol Connectors_kl:CONN_40
Connections:
- new net +IPS: C?.1, C?.1, DA?.1 (IN), L?.1
- new net +VCCIO3V3: C?.1, DD1.U16 (VCC-PD), L?.2
- new net +VDD_LCD: C?.1, L?.1, TP?.1, XL?.4
- new net GND: C?.1, C?.2, C?.2, C?.2, C?.2, DA?.2 (GND), R?.2, R?.2, XL?.13, XL?.14, XL?.21, XL?.22, XL?.29, XL?.3, XL?.36, XL?.5, XL?.6, XL?.PAD
- new net LCDLX: D?.A, DA?.5 (SW), L?.2
- new net LCD_DISP: DD1.Y14 (PD24), TP?.1, XL?.31
- new net LCD_PWM: DA?.3 (EN), DD1.Y13 (PD22/PWM0/MDC), R?.1
- new net LCD_XL: XL?.39
- new net LCD_XR: XL?.37
- new net LCD_YD: XL?.38
- new net LCD_YU: XL?.40
- new net LTDC_B2: DD1.AC16 (PD12/LCD-D18/LVDS-VP0/RGMII-RXCK/RMII-NULL), XL?.23
- new net LTDC_B3: DD1.AB16 (PD13/LCD-D19/LVDS-VN0/RGMII-RXCTL/RMII-CRS-DV), XL?.24
- new net LTDC_B4: DD1.AB15 (PD14/LCD-D20/LVDS-VP1/RGMII-NULL/RMII-RXER), XL?.25
- new net LTDC_B5: DD1.AB14 (PD15/LCD-D21/LVDS-VN1/RGMII-TXD3/RMII-NULL/CCIR-D6), XL?.26
- new net LTDC_B6: DD1.AC14 (PD16/LCD-D22/LVDS-VP2/RGMII-TXD2/RMII-NULL/CCIR-D7), XL?.27
- new net LTDC_B7: DD1.AC13 (PD17/LCD-D23/LVDS-VN2/RGMII-TXD1/RMII-TXD1), XL?.28
- new net LTDC_CLK: DD1.AB13 (PD18/LCD-CLK/LVDS-VPC/RGMII-TXD0/RMII-TXD0), TP?.1, XL?.30
- new net LTDC_DE: DD1.AB12 (PD19/LCD-DE/LVDS-VNC/RGMII-TXCK/RMII-TXCK), TP?.1, XL?.34
- new net LTDC_G2: DD1.Y11 (PD6/LCD-D10/CCIR-D2), XL?.15
- new net LTDC_G3: DD1.AA16 (PD7/LCD-D11/CCIR-D3), XL?.16
- new net LTDC_G4: DD1.V17 (PD8/LCD-D12/RGMII-RXD3/RMII-NULL/CCIR-D4), XL?.17
- new net LTDC_G5: DD1.AA13 (PD9/LCD-D13/RGMII-RXD2/RMII-NULL/CCIR-D5), XL?.18
- new net LTDC_G6: DD1.W16 (PD10/LCD-D14/RGMII-RXD1/RMII-RXD1), XL?.19
- new net LTDC_G7: DD1.Y16 (PD11/LCD-D15/RGMII-RXD0/RMII-RXD0), XL?.20
- new net LTDC_HSYNC: DD1.AB11 (PD20/LCD-HSYNC/LVDS-VP3/RGMII-TXCTL/RMII-TXEN), TP?.1, XL?.32
- new net LTDC_R2: DD1.AA20 (PD0/LCD-D2/UART3-TX/SPI1-CS/CCIR-CLK), XL?.7
- new net LTDC_R3: DD1.AA17 (PD1/LCD-D3/UART3-RX/SPI1-CLK/CCIR-DE), XL?.8
- new net LTDC_R4: DD1.W19 (PD2/LCD-D4/UART4-TX/SPI1-MOSI/CCIR-HSYNC), XL?.9
- new net LTDC_R5: DD1.AA14 (PD3/LCD-D5/UART4-RX/SPI1-MISO/CCIR-VSYNC), XL?.10
- new net LTDC_R6: DD1.V18 (PD4/LCD-D6/UART4-RTS/CCIR-D0), XL?.11
- new net LTDC_R7: DD1.AA15 (PD5/LCD-D7/UART4-CTS/CCIR-D1), XL?.12
- new net LTDC_VSYNC: DD1.AC11 (PD21/LCD-VSYNC/LVDS-VN3/RGMII-CLKIN/RMII-NULL), TP?.1, XL?.33
- new net VLED+: C?.2, D?.C, XL?.2
- new net VLED-: DA?.4 (FB), R?.1, XL?.1
- no-connect marks 0 -> 2
Other:
- note added: "20R => 15mA 15R => 20mA"
- note added: "25+ v here"
- note added: "NC"
- note added: "RGB666 is implemented here. CPU has 18 bit RGB only."

Commit message: Before eMMC removing
Parts:
- added C? (x2): 0u1, Capacitors:CAP_0402, symbol Tittar_kl:C
- added C?: 10u, Capacitors:CAP_0603, symbol Tittar_kl:C
- added DD?: XPT2046, SO_DIL_TSSOP:TSSOP16, symbol Sensors:XPT2046
- added R?: 47k, Resistors:RES_0603, symbol Tittar_kl:R
Connections:
- net +VCCIO3V3: now also C?.1, C?.1, DD?.1 (VCC), DD?.10 (IOVDD), R?.1
- net GND: now also C?.2, C?.2, C?.2, DD?.6 (GND)
- net LCD_XL: now also DD?.4 (XN)
- net LCD_XR: now also DD?.2 (XP)
- net LCD_YD: now also DD?.3 (YP)
- net LCD_YU: now also DD?.5 (YN)
- new net: C?.1, DD?.9 (VREF)
- new net TCH.BUSY: DD?.13 (BUSY)
- new net TCH.CS: DD?.15 (~{CS})
- new net TCH.IRQ: DD?.11 (~{PENIRQ}), R?.2
- new net TCH.MISO: DD?.12 (DOUT)
- new net TCH.MOSI: DD?.14 (DIN)
- new net TCH.SCK: DD?.16 (DCLK)
- no-connect marks 2 -> 4
Other:
- note added: "Touch Controller"
- moved on the sheet: C?, D?, DA?, DD1H, L?, R?, TP?, XL?
