File: PCB/WiFiBt.kicad_sch (KiCad schematic)
At the start: 0 parts

Commit message: Before eMMC removing
Parts:
- added DD1: A64, BGA:BGA-529_23x23_15.0x15.0mm, symbol Allwinner:A64
Changed lines of the file:
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@@
 (kicad_sch (version 20211123) (generator eeschema)
   (paper "A4")
+  (symbol (lib_id "Allwinner:A64") (at 82.55 68.58 0) (unit 11)
+    (in_bom yes) (on_board yes) (fields_autoplaced)
+    (property "Reference" "DD1" (id 0) (at 66.04 63.5 0))
+    (property "Value" "A64" (id 1) (at 66.04 66.04 0))
+    (property "Footprint" "BGA:BGA-529_23x23_15.0x15.0mm" (id 2) (at 82.55 60.96 0)
+      (effects (font (size 1.27 1.27)) hide)
+    )
+    (property "Datasheet" "" (id 3) (at 82.55 68.58 0)
+      (effects (font (size 1.27 1.27)) hide)
+    )
+    (pin "AB17")
+    (pin "AB18")
+    (pin "AB19")
+    (pin "AC17")
+    (pin "AC19")
+    (pin "T17")
+    (pin "U19")
+    (pin "U20")
+    (pin "U21")
+    (pin "U22")
+    (pin "U23")
+    (pin "V21")
+    (pin "V22")
+    (pin "W23")
+    (pin "Y21")
+  )
 )
