File: PCB/uSD.kicad_sch (KiCad schematic)
At the start: 0 parts

Commit message: Before eMMC removing
Parts:
- added C?: 10u, Capacitors:CAP_0603, symbol Tittar_kl:C
- added DD?: A64, BGA:BGA-529_23x23_15.0x15.0mm, symbol Allwinner:A64
- added R?: 10k, Resistors:RES_0402_sm, symbol Tittar_kl:R
- added R?: 33R, Resistors:RES_0402_sm, symbol Tittar_kl:R
- added XL?: CONN_MICROSD, Installation:MICROSD_CAP_FIX05A, symbol Connectors_kl:CONN_MICROSD
Connections:
- new net: DD?.AC8 (PF2/SDC0-CLK/UART0-TX), R?.2
- new net +VCCIO3V3: C?.1, R?.2, XL?.4 (VDD)
- new net GND: C?.2, XL?.6 (GND), XL?.H (Housing)
- new net SD_CLK: R?.1, XL?.5 (SCK/CLK)
- new net SD_CMD: DD?.W9 (PF3/SDC0-CMD/JTAG-DO1), R?.1, XL?.3 (MOSI/CMD)
- new net SD_DAT0: DD?.W13 (PF1/SDC0-D0/JTAG-DI1), XL?.7 (MISO/DAT0)
- new net SD_DAT1: DD?.AB10 (PF0/SDC0-D1/JTAG-MS1), XL?.8 (DAT1)
- new net SD_DAT2: DD?.AB9 (PF5/SDC0-D2/JTAG-CK1), XL?.1 (DAT2)
- new net SD_DAT3: DD?.AB6 (PF4/SDC0-D3/UART0-RX), XL?.2 (~{SS}/DAT3)
- no-connect marks 0 -> 1
